Commit message: Update rplidar.urdf.xacro

File: gobilda_ws/src/gobilda_robot/description/urdf/sensors/rplidar.urdf.xacro (robot description, xacro)
@@ -18,5 +18,5 @@
     <visual>
       <geometry>
-        <mesh filename="package://turtlebot4_description/meshes/rplidar.dae" scale="1 1 1" />
+        <mesh filename="package://gobilda_robot/description/meshes/rplidar.dae" scale="1 1 1" />
       </geometry>
     </visual>
