Commit message: Update oakd.urdf.xacro

File: gobilda_ws/src/gobilda_robot/description/urdf/sensors/oakd.urdf.xacro (robot description, xacro)
@@ -2,5 +2,4 @@
 <robot xmlns:xacro="http://ros.org/wiki/xacro">
 <xacro:macro name="oakd" params="name:=oakd parent_link *origin model:=pro">
-  <xacro:include filename="$(find irobot_create_description)/urdf/common_properties.urdf.xacro"/>
   <xacro:property name="mass"       value="0.061"/>
   <xacro:property name="baseline" value="0.075" />
@@ -22,5 +21,5 @@
     <visual>
       <geometry>
-        <mesh filename="package://turtlebot4_description/meshes/${name}_${model}.dae" scale="1 1 1" />
+        <mesh filename="package://gobilda_robot/description/meshes/${name}_${model}.dae" scale="1 1 1" />
       </geometry>
     </visual>
