Commit message: Update gobilda.urdf.xacro

File: gobilda_ws/src/gobilda_robot/description/urdf/gobilda.urdf.xacro (robot description, xacro)
@@ -2,8 +2,25 @@
 <robot xmlns:xacro="http://www.ros.org/wiki/xacro" name="diffdrive_robot">
   <xacro:arg name="prefix" default="" />
+  <xacro:arg name="gazebo" default="false" />
   <xacro:arg name="use_mock_hardware" default="false" />
+  <xacro:property name="rplidar_x_offset"              value="${-4*cm2m}"/>
+  <xacro:property name="rplidar_y_offset"              value="${0*cm2m}"/>
+  <xacro:property name="rplidar_z_offset"              value="${9.8715*cm2m}"/>
+  <xacro:property name="oakd_pro_x_offset"             value="${5.84*cm2m}"/>
+  <xacro:property name="oakd_pro_y_offset"             value="${0*cm2m}"/>
+  <xacro:property name="oakd_pro_z_offset"             value="${9.676*cm2m}"/>
   <xacro:include filename="$(find gobilda_robot)/urdf/gobilda_description.urdf.xacro" />
   <xacro:include filename="$(find gobilda_robot)/ros2_control/gobilda.ros2_control.xacro" />
+  <!-- Adding files for the sensors on the robot -->
+  <xacro:include filename="$(find gobilda_robot)/urdf/sensors/rplidar.urdf.xacro" />
+  <xacro:include filename="$(find gobilda_robot)/urdf/sensors/oakd.urdf.xacro" />
   <xacro:gobilda_robot prefix="$(arg prefix)" />
   <xacro:gobilda_ros2_control name="Gobilda" prefix="$(arg prefix)" use_mock_hardware="$(arg use_mock_hardware)"/>
+  <!-- Gobilda sensor definitions -->
+  <xacro:rplidar name="rplidar" parent_link="base_link" gazebo="$(arg gazebo)">
+    <origin xyz="${rplidar_x_offset} ${rplidar_y_offset} ${rplidar_z_offset}"/>
+  </xacro:rplidar>
+  <xacro:oakd model="pro" parent_link="base_link">
+    <origin xyz="${oakd_pro_x_offset} ${oakd_pro_y_offset} ${oakd_pro_z_offset}"/>
+  </xacro:oakd>
 </robot>

Commit message: Fixed some of the directory structure that was missing or incorrect

File: gobilda_ws/src/gobilda_robot/description/urdf/gobilda.urdf.xacro (robot description, xacro)
@@ -2,25 +2,8 @@
 <robot xmlns:xacro="http://www.ros.org/wiki/xacro" name="diffdrive_robot">
   <xacro:arg name="prefix" default="" />
-  <xacro:arg name="gazebo" default="false" />
   <xacro:arg name="use_mock_hardware" default="false" />
-  <xacro:property name="rplidar_x_offset"              value="${-4*cm2m}"/>
-  <xacro:property name="rplidar_y_offset"              value="${0*cm2m}"/>
-  <xacro:property name="rplidar_z_offset"              value="${9.8715*cm2m}"/>
-  <xacro:property name="oakd_pro_x_offset"             value="${5.84*cm2m}"/>
-  <xacro:property name="oakd_pro_y_offset"             value="${0*cm2m}"/>
-  <xacro:property name="oakd_pro_z_offset"             value="${9.676*cm2m}"/>
-  <xacro:include filename="$(find gobilda_robot)/urdf/gobilda_description.urdf.xacro" />
-  <xacro:include filename="$(find gobilda_robot)/ros2_control/gobilda.ros2_control.xacro" />
-  <!-- Adding files for the sensors on the robot -->
-  <xacro:include filename="$(find gobilda_robot)/urdf/sensors/rplidar.urdf.xacro" />
-  <xacro:include filename="$(find gobilda_robot)/urdf/sensors/oakd.urdf.xacro" />
-  <xacro:gobilda_robot prefix="$(arg prefix)" />
+  <xacro:include filename="$(find gobilda_robot)/urdf/gobilda_description.urdf.xacro"/>
+  <xacro:include filename="$(find gobilda_robot)/ros2_control/gobilda.ros2_control.xacro"/>
+  <xacro:gobilda_robot prefix="$(arg prefix)"/>
   <xacro:gobilda_ros2_control name="Gobilda" prefix="$(arg prefix)" use_mock_hardware="$(arg use_mock_hardware)"/>
-  <!-- Gobilda sensor definitions -->
-  <xacro:rplidar name="rplidar" parent_link="base_link" gazebo="$(arg gazebo)">
-    <origin xyz="${rplidar_x_offset} ${rplidar_y_offset} ${rplidar_z_offset}"/>
-  </xacro:rplidar>
-  <xacro:oakd model="pro" parent_link="base_link">
-    <origin xyz="${oakd_pro_x_offset} ${oakd_pro_y_offset} ${oakd_pro_z_offset}"/>
-  </xacro:oakd>
 </robot>

File: gobilda_ws/src/gobilda_robot/description/urdf/gobilda_description.urdf.xacro (robot description, xacro)
@@ -2,104 +2,130 @@
 <robot xmlns:xacro="http://www.ros.org/wiki/xacro">
   <xacro:macro name="gobilda_robot" params="prefix">
-  <!-- Constants for robot dimensions -->
-  <xacro:property name="PI" value="3.1415926535897931"/>
-  <xacro:property name="base_mass" value="0.3" /> <!-- arbitrary value for base mass -->
-  <xacro:property name="base_width" value="0.1" />
-  <xacro:property name="base_length" value="0.1" />
-  <xacro:property name="base_height" value="0.05" />
-  <xacro:property name="wheel_mass" value="0.3" /> <!-- arbitrary value for wheel mass -->
-  <xacro:property name="wheel_len" value="0.020" />
-  <xacro:property name="wheel_radius" value="0.015" />
-  <xacro:property name="z_offset" value="-${base_height/2}" /> <!-- Space btw top of beam and the each joint -->
-  <!-- Base Link -->
-  <link name="base_link">
-    <collision>
-      <origin xyz="0 0 0" rpy="0 0 0"/>
-      <geometry>
-        <box size="${base_width} ${base_length} ${base_height}"/>
-      </geometry>
-    </collision>
-    <visual>
-      <origin xyz="0 0 ${base_height/2}" rpy="0 0 0"/>
-      <geometry>
-        <box size="${base_width} ${base_length} ${base_height}"/>
-      </geometry>
-    </visual>
-    <!--
-    <inertial>
-      <origin xyz="0 0 0" rpy="0 0 0"/>
-      <mass value="${base_mass}"/>
-      <inertia
-        ixx="${base_mass / 12.0 * (base_length*base_length + base_height*base_height)}" ixy="0.0" ixz="0.0"
-        iyy="${base_mass / 12.0 * (base_height*base_height + base_width*base_width)}" iyz="0.0"
-        izz="${base_mass / 12.0 * (base_width*base_width + base_length*base_length)}"/>
-      </inertial> -->
-  </link>
-  <joint name="left_wheel_joint" type="continuous">
-    <parent link="base_link"/>
-    <child link="left_wheel"/>
-    <origin xyz="0 -${base_width/2} ${z_offset}" rpy="0 0 0"/>
-    <axis xyz="0 1 0"/>
-    <dynamics damping="0.2"/>
-    <limit effort="100" velocity="1.0"/>
-  </joint>
-  <!-- left wheel Link -->
-  <link name="left_wheel">
-    <collision>
-      <origin xyz="0 0 0" rpy="${PI/2} 0 0"/>
-      <geometry>
-        <cylinder length="${wheel_len}" radius="${wheel_radius}"/>
-      </geometry>
-    </collision>
-    <visual>
-      <origin xyz="0 0 0" rpy="${PI/2} 0 0"/>
-      <geometry>
-        <cylinder length="${wheel_len}" radius="${wheel_radius}"/>
-      </geometry>
-    </visual>
-    <!--
-    <inertial>
-      <origin xyz="0 0 0" rpy="${PI/2} 0 0"/>
-      <mass value="${wheel_mass}"/>
-      <inertia
-        ixx="${wheel_mass / 12.0 * (3*wheel_radius*wheel_radius + wheel_len*wheel_len)}" ixy="0.0" ixz="0.0"
-        iyy="${wheel_mass / 12.0 * (3*wheel_radius*wheel_radius + wheel_len*wheel_len)}" iyz="0.0"
-        izz="${wheel_mass / 2.0 * wheel_radius*wheel_radius}"/>
-      </inertial>
-      -->
-  </link>
-  <joint name="right_wheel_joint" type="continuous">
-    <parent link="base_link"/>
-    <child link="right_wheel"/>
-    <origin xyz="0 ${base_width/2} ${z_offset}" rpy="0 0 0"/>
-    <axis xyz="0 1 0"/>
-    <dynamics damping="0.2"/>
-    <limit effort="100" velocity="1.0"/>
-  </joint>
-  <!-- right wheel Link -->
-  <link name="right_wheel">
-    <collision>
-      <origin xyz="0 0 0" rpy="${PI/2} 0 0"/>
-      <geometry>
-        <cylinder length="${wheel_len}" radius="${wheel_radius}"/>
-      </geometry>
-    </collision>
-    <visual>
-      <origin xyz="0 0 0" rpy="${PI/2} 0 0"/>
-      <geometry>
-        <cylinder length="${wheel_len}" radius="${wheel_radius}"/>
-      </geometry>
-    </visual>
-    <!--
-    <inertial>
-      <origin xyz="0 0 0" rpy="${PI/2} 0 0"/>
-      <mass value="${wheel_mass}"/>
-      <inertia
-        ixx="${wheel_mass / 12.0 * (3*wheel_radius*wheel_radius + wheel_len*wheel_len)}" ixy="0.0" ixz="0.0"
-        iyy="${wheel_mass / 12.0 * (3*wheel_radius*wheel_radius + wheel_len*wheel_len)}" iyz="0.0"
-        izz="${wheel_mass / 2.0 * wheel_radius*wheel_radius}"/>
-      </inertial>
-      -->
-  </link>
-  </xacro:macro>
+    <!-- Robot Parameters -->
+    <xacro:property name="PI" value="3.14159265"/>
+    <xacro:property name="body_length" value="0.5"/>
+    <xacro:property name="body_width" value="0.3"/>
+    <xacro:property name="body_height" value="0.1"/>
+    <xacro:property name="body_density" value="7850.0"/> <!-- Steel -->
+    <xacro:property name="body_mass" value="${body_density * body_length * body_height * body_width}"/>
+    <xacro:property name="body_inertia_x" value="${1.0/12.0 * body_mass * (body_height*body_height + body_width*body_width)}"/>
+    <xacro:property name="body_inertia_y" value="${1.0/12.0 * body_mass * (body_length*body_length + body_height*body_height)}"/>
+    <xacro:property name="body_inertia_z" value="${1.0/12.0 * body_mass * (body_length*body_length + body_width*body_width)}"/>
+    <xacro:property name="wheel_radius" value="0.06"/>
+    <xacro:property name="wheel_width" value="0.05"/>
+    <xacro:property name="wheel_separation" value="${body_width + wheel_width}"/>
+    <xacro:property name="wheel_offset_x" value="0.1"/>
+    <xacro:property name="wheel_offset_y" value="0.09"/>
+    <xacro:property name="wheel_density" value="900"/> <!-- Ruber -->
+    <xacro:property name="wheel_mass" value="${wheel_density * PI * wheel_radius * wheel_radius * wheel_width}"/>
+    <xacro:property name="wheel_inertia_x" value="${1.0/12.0 * wheel_mass * (3*wheel_radius*wheel_radius + wheel_width*wheel_width)}"/>
+    <xacro:property name="wheel_inertia_y" value="${1.0/12.0 * wheel_mass * (3*wheel_radius*wheel_radius + wheel_width*wheel_width)}"/>
+    <xacro:property name="wheel_inertia_z" value="${1.0/2.0 * wheel_mass * wheel_radius * wheel_radius}"/>
+    <xacro:property name="lidar_offset_x" value="0.1"/>
+    <xacro:property name="lidar_offset_y" value="0.0"/>
+    <xacro:property name="lidar_offset_z" value="0.03"/>
+    <!-- Control Parameters -->
+    <xacro:property name="max_linear_acceleration" value="10"/>
+    <!-- Links -->
+    <!-- Body Link -->
+    <link name="base_link">
+        <visual>
+            <origin xyz="0.0 0.0 0.0" rpy="0.0 0.0 0.0"/>
+            <geometry>
+                <box size="${body_length} ${body_width} ${body_height}"/>
+            </geometry>
+        </visual>
+        <collision>
+            <origin xyz="0.0 0.0 0.0" rpy="0.0 0.0 0.0"/>
+            <geometry>
+                <box size="${body_length} ${body_width} ${body_height}"/>
+            </geometry>
+        </collision>
+        <inertial>
+            <mass value="10"/>
+            <inertia ixx="${body_inertia_x}" ixy="0.0" ixz="0.0" iyy="${body_inertia_y}" iyz="0" izz="${body_inertia_z}"/>
+            <origin xyz="0 0 0" rpy="0 0 0"/>
+        </inertial>
+    </link>
+    <!-- Left Wheel -->
+    <link name="left_wheel_link">
+        <visual>
+            <origin xyz="-${wheel_offset_x} 0.27 -0.01" rpy="0 0 0"/>
+            <geometry>
+                <sphere radius="${wheel_radius}"/>
+            </geometry>
+        </visual>
+        <collision>
+            <origin xyz="-${wheel_offset_x} 0.27 -0.01" rpy="0 0 0"/>
+            <geometry>
+                <sphere radius="${wheel_radius}" length="${wheel_width}"/>
+            </geometry>
+        </collision>
+        <inertial>
+            <mass value="2"/>
+            <inertia ixx="${wheel_inertia_x}" ixy="0.0" ixz="0.0" iyy="${wheel_inertia_y}" iyz="0" izz="${wheel_inertia_z}"/>
+            <origin xyz="0.0 0.0 0.0" rpy="1.570795 0.0 0.0"/>
+        </inertial>
+    </link>
+    <!-- Right Wheel -->
+    <link name="right_wheel_link">
+        <visual>
+            <origin xyz="-${wheel_offset_x} -${wheel_offset_y} -0.01" rpy="0 0 0"/>
+            <geometry>
+                <sphere radius="${wheel_radius}" />
+            </geometry>
+        </visual>
+        <collision>
+            <origin xyz="-${wheel_offset_x} -${wheel_offset_y} -0.01" rpy="0 0 0"/>
+            <geometry>
+                <sphere radius="${wheel_radius}"/>
+            </geometry>
+        </collision>
+        <inertial>
+            <mass value="2"/>
+            <inertia ixx="${wheel_inertia_x}" ixy="0.0" ixz="0.0" iyy="${wheel_inertia_y}" iyz="0" izz="${wheel_inertia_z}"/>
+            <origin xyz="0.0 0.0 0.0" rpy="1.570795 0.0 0.0"/>
+        </inertial>
+    </link>
+    <!-- Laser -->
+    <link name="laser">
+        <visual>
+            <origin xyz="${lidar_offset_x} ${lidar_offset_y} ${lidar_offset_z}" rpy="0 0 0"/>
+            <geometry>
+                <box size="0.05 0.05 0.05"/>
+            </geometry>
+        </visual>
+        <collision>
+            <origin xyz="${lidar_offset_x} ${lidar_offset_y} ${lidar_offset_z}" rpy="0 0 0"/>
+            <geometry>
+                <box size="0.05 0.05 0.05"/>
+            </geometry>
+        </collision>
+    </link>
+    <!-- Joints -->
+    <!-- Left Wheel Joint -->
+    <joint name="left_wheel_joint" type="continuous">
+        <origin xyz="-${wheel_offset_x} ${-wheel_offset_y} 0" rpy="0 0 0"/>
+        <parent link="base_link"/>
+        <child link="left_wheel_link"/>
+        <axis xyz="0 1 0"/>
+        <limit effort="100" velocity="10.0"/>
+        <dynamics damping="0.1" friction="0.1"/>
+    </joint>
+    <!-- Right Wheel Joint -->
+    <joint name="right_wheel_joint" type="continuous">
+        <origin xyz="-${wheel_offset_x} ${-wheel_offset_y} 0" rpy="0 0 0"/>
+        <parent link="base_link"/>
+        <child link="right_wheel_link"/>
+        <axis xyz="0 1 0"/>
+        <limit effort="100" velocity="10.0"/>
+        <dynamics damping="0.1" friction="0.1"/>
+    </joint>
+    <!-- Lidar Joint (fixed) -->
+    <joint name="lidar_joint" type="fixed">
+        <origin xyz="${lidar_offset_x} ${lidar_offset_y} ${lidar_offset_z}" rpy="0 0 0"/>
+        <parent link="base_link"/>
+        <child link="laser"/>
+    </joint>
+</xacro:macro>
 </robot>
