Commit message: Working version of the code where: VI-Odom working with oakd, ICP working with rplidar, EFK-odom work with robot_localization. Deleted the JETGPIO library and added sys/class calls inside the ros2_control thread. Debatable whether this is correct for not. Acutal control of the robot when running ROS2 is very jittery. TODO: Add scripts for setting up Orin/Jetpack environment!

File: gobilda_ws/src/gobilda_robot/description/urdf/gobilda_description.urdf.xacro (robot description, xacro)
@@ -156,9 +156,12 @@
      <!-- From Turtlebot4 package sensor definitions -->
     <xacro:rplidar name="rplidar" parent_link="base_link" gazebo="$(arg gazebo)">
+        <!-- Should correspond to the actual offset on the robot -->
         <origin xyz="${lidar_offset_x} ${lidar_offset_y} ${lidar_offset_z}"
-                rpy="0 0 0"/>
+                rpy="0 0 -0.15"/>
     </xacro:rplidar>
     <xacro:oakd model="pro" parent_link="base_link">
-        <origin xyz="${oakd_pro_x_offset} ${oakd_pro_y_offset} ${oakd_pro_z_offset}"/>
+        <!-- Should correspond to the actual offset on the robot -->
+        <origin xyz="${oakd_pro_x_offset} ${oakd_pro_y_offset} ${oakd_pro_z_offset}"
+                rpy="0 0 0"/>
     </xacro:oakd>
 </xacro:macro>

Commit message: Refactoring code for new assignments.

File: gobilda_ws/src/gobilda_robot/description/urdf/gobilda_description.urdf.xacro (robot description, xacro)
@@ -26,10 +26,10 @@
     <xacro:property name="wheel_inertia_y" value="${1.0/12.0 * wheel_mass * (3*wheel_radius*wheel_radius + wheel_width*wheel_width)}"/>
     <xacro:property name="wheel_inertia_z" value="${1.0/2.0 * wheel_mass * wheel_radius * wheel_radius}"/>
-    <xacro:property name="lidar_offset_x" value="0.1"/>
-    <xacro:property name="lidar_offset_y" value="0.0"/>
-    <xacro:property name="lidar_offset_z" value="0.07"/>
-    <xacro:property name="oakd_pro_x_offset"             value="0.11"/>
-    <xacro:property name="oakd_pro_y_offset"             value="0.1"/>
-    <xacro:property name="oakd_pro_z_offset"             value="0.07"/>
+    <xacro:property name="lidar_offset_x"   value="0.1"/>
+    <xacro:property name="lidar_offset_y"   value="-0.1"/>
+    <xacro:property name="lidar_offset_z"   value="0.07"/>
+    <xacro:property name="oakd_pro_x_offset"    value="0.2"/>
+    <xacro:property name="oakd_pro_y_offset"    value="0.1"/>
+    <xacro:property name="oakd_pro_z_offset"    value="0.07"/>
     <!-- Control Parameters -->
     <xacro:property name="max_linear_acceleration" value="10"/>
@@ -82,5 +82,5 @@
             <inertia ixx="${wheel_inertia_x}" ixy="0" ixz="0"
                      iyy="${wheel_inertia_y}" iyz="0" izz="${wheel_inertia_z}"/>
-            </inertial>
+        </inertial>
     </link>
     <!-- Left Wheel Joint and Link Front-->
@@ -103,4 +103,10 @@
             </geometry>
         </collision>
+        <inertial>
+            <mass value="2"/>
+            <origin xyz="0 0 0" rpy="0 0 0"/>
+            <inertia ixx="${wheel_inertia_x}" ixy="0" ixz="0"
+                     iyy="${wheel_inertia_y}" iyz="0" izz="${wheel_inertia_z}"/>
+        </inertial>
     </link>
     <!-- Right Wheel Joint & Link Rear -->
@@ -153,4 +159,10 @@
             </geometry>
         </collision>
+        <inertial>
+            <mass value="2"/>
+            <origin xyz="0 0 0" rpy="0 0 0"/>
+            <inertia ixx="${wheel_inertia_x}" ixy="0" ixz="0"
+                     iyy="${wheel_inertia_y}" iyz="0" izz="${wheel_inertia_z}"/>
+        </inertial>
     </link>
      <!-- From Turtlebot4 package sensor definitions -->
@@ -158,5 +170,5 @@
         <!-- Should correspond to the actual offset on the robot -->
         <origin xyz="${lidar_offset_x} ${lidar_offset_y} ${lidar_offset_z}"
-                rpy="0 0 -0.15"/>
+                rpy="0 0 0.30"/>
     </xacro:rplidar>
     <xacro:oakd model="pro" parent_link="base_link">
@@ -165,4 +177,4 @@
                 rpy="0 0 0"/>
     </xacro:oakd>
-</xacro:macro>
+  </xacro:macro>
 </robot>
